File: pcb/C128-keyboard.kicad_sch (KiCad schematic)
At the start: 104 parts, among them CN1 C128, CN2 Neo128, SW1 Inst/Del, SW10 Esc, SW11 Alt, SW12 Return, SW13 W, SW14 R, SW15 Y, SW16 I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

Commit message: Wiring fixes for latch keys
Connections:
- net 40_80: now also SW92.4 (LEDGND)
- net CAPLK: now also SW91.4 (LEDGND), U1.4 (~{OUT}); no longer U1.5 (OUT)
- net at U2.5 (OUT): no longer SW92.4 (LEDGND)
