File: pcb/C128-keyboard.kicad_pcb (KiCad board)
At the start: 2 copper layers, 395 x 132 mm, 103 parts, among them CN2 Neo128, SW1 Inst/Del, SW10 Esc, SW11 Alt, SW12 Return, SW13 W, SW14 R, SW15 Y, SW16 I, SW17 P, SW18 *, SW19 LeftArrow, SW2 3, SW20 Num8, SW21 Num+, SW22 Num0, SW23 Crsr Horiz, SW24 A, SW25 D, SW26 G, SW27 J, SW28 L, SW29 ;, SW3 5, SW30 Ctrl, SW31 Num5, SW32 Num-, SW33 Num., SW34 F7, SW35 4, SW36 6, SW37 8, SW38 0, SW39 -, SW4 7, SW40 Clr/Home, SW41 2, SW42 Tab, SW43 LineFeed, SW44 Crsr-Up, SW45 F1, SW46 Z, SW47 C, SW48 B, SW49 M, SW5 9, SW50 ., SW51 R-Shift, SW52 Space, SW53 Num2, SW54 NumEnter, SW55 Crsr-Down, SW56 F3, SW57 S, SW58 F, SW59 H, SW6 +, SW60 K, SW61 :, SW62 =, SW63 C=, SW64 Num4, SW65 Num6, SW66 Crsr-Left, SW67 F5, SW68 E, SW69 T, SW7 £, SW70 U, SW71 O, SW72 @, SW73 UpArrow, SW74 Q, SW75 Num7, SW76 Num9, SW77 Crsr-Right, SW78 Crsr Vert, SW79 L-Shift, SW8 1, SW80 X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

Commit message: Wiring fixes for latch keys
Parts:
- moved SW34 0.67 mm to (494.5, 90.2)
- moved SW56 0.67 mm to (456.4, 90.2)
- moved SW67 0.67 mm to (475.4, 90.2)
- moved SW45 0.67 mm to (437.3, 90.2)
- moved R1 0.46 mm to (170.3, 95.3)
- moved SW10 0.46 mm to (118.3, 90.2)
- moved SW11 0.46 mm to (156.4, 90.2)
- moved SW42 0.46 mm to (137.3, 90.2)
- moved SW91 0.46 mm to (175.4, 90.2)
- moved SW44 0.44 mm to (346.9, 90.2)
- moved SW55 0.44 mm to (365.9, 90.2)
- moved SW66 0.44 mm to (385.0, 90.2)
- moved SW77 0.44 mm to (404.0, 90.2)
- moved R2 0.41 mm to (265.7, 95.3)
- moved U2 0.41 mm to (277.2, 95.7)
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Connections:
- SW91 pad 4: Net-(SW91-Pad4) -> CAPLK
- SW92 pad 4: Net-(SW92-Pad4) -> 40_80
- U1 pad 4: Net-(SW91-Pad4) -> CAPLK
- U1 pad 5: CAPLK -> (no net)
- U2 pad 5: Net-(SW92-Pad4) -> (no net)
Routing:
- net Net-(SW91-Pad4): track 10.8 -> 0.00 mm
- net CAPLK: track 193.7 -> 203.0 mm
- net 40_80: track 77.6 -> 85.5 mm
- net Net-(SW92-Pad4): track 6.36 -> 0.00 mm
- net Net-(R2-Pad1): track 2.73 -> 3.39 mm
- net ROW4: track 585.2 -> 584.6 mm
Other:
- board size 395 x 132 mm -> 395.1 x 132 mm

Commit message: Adding pad for plate grounding strap
Parts:
- added Plate Ground: MountingHole_3.2mm_M3_Pad_Via, MountingHole:MountingHole_3.2mm_M3_Pad_Via, F.Cu at (216.3, 80.4)
Changed lines of the file:
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@@
+		(embedded_fonts no)
+	)
+	(footprint "MountingHole:MountingHole_3.2mm_M3_Pad_Via"
+		(layer "F.Cu")
+		(at 216.252944 80.377944)
+		(descr "Mounting Hole 3.2mm, M3, generated by kicad-footprint-generator mountinghole.py")
+		(tags "mountinghole M3")
+		(property "Reference" "Plate Ground"
+			(at 0 -4.15 0)
+			(layer "B.SilkS")
+			(effects
+				(font
+					(size 1 1)
+					(thickness 0.15)
+				)
+			)
+		)
+		(property "Value" "MountingHole_3.2mm_M3_Pad_Via"
+			(at 0 4.15 0)
+			(layer "F.Fab")
+			(effects
+				(font
+					(size 1 1)
+					(thickness 0.15)
+				)
+			)
+		)
+		(property "Datasheet" ""
+			(at 0 0 0)
+			(layer "F.Fab")
+			(hide yes)
+			(effects
+				(font
+					(size 1.27 1.27)
+					(thickness 0.15)
+				)
+			)
+		)
+		(property "Description" ""
+			(at 0 0 0)
+			(layer "F.Fab")
+			(hide yes)
+			(effects
+				(font
+					(size 1.27 1.27)
+					(thickness 0.15)
+				)
+			)
+		)
+		(attr exclude_from_pos_files exclude_from_bom)
+		(fp_circle
+			(center 0 0)
+			(end 3.2 0)
+			(stroke
+				(width 0.15)
+				(type solid)
+			)
+			(fill no)
+			(layer "Cmts.User")
+		)
+		(fp_circle
+			(center 0 0)
+			(end 3.45 0)
+			(stroke
+				(width 0.05)
+				(type solid)
+			)
+			(fill no)
+			(layer "F.CrtYd")
+		)
+		(fp_text user "${REFERENCE}"
+			(at 0 0 0)
+			(layer "F.Fab")
+			(effects
+				(font
+					(size 1 1)
+					(thickness 0.15)
+				)
+			)
+		)
+		(pad "1" thru_hole circle
+			(at -2.4 0)
+			(size 0.8 0.8)
+			(drill 0.5)
+			(layers "*.Cu" "*.Mask")
+			(remove_unused_layers no)
+			(net 1 "GND")
+			(zone_connect 2)
+		)
+		(pad "1" thru_hole circle
+			(at -1.697056 -1.697056)
+			(size 0.8 0.8)
+			(drill 0.5)
+			(layers "*.Cu" "*.Mask")
+			(remove_unused_layers no)
+			(net 1 "GND")
+			(zone_connect 2)
+		)
+		(pad "1" thru_hole circle
+			(at -1.697056 1.697056)
+			(size 0.8 0.8)
+			(drill 0.5)
+			(layers "*.Cu" "*.Mask")
+			(remove_unused_layers no)
+			(net 1 "GND")
+			(zone_connect 2)
+		)
+		(pad "1" thru_hole circle
+			(at 0 -2.4)
+			(size 0.8 0.8)
+			(drill 0.5)
+			(layers "*.Cu" "*.Mask")
+			(remove_unused_layers no)
+			(zone_connect 2)
+		)
+		(pad "1" thru_hole circle
+			(at 0 0)
+			(size 6.4 6.4)
+			(drill 3.2)
+			(layers "*.Cu" "*.Mask")
+			(remove_unused_layers no)
+			(net 1 "GND")
+			(zone_connect 2)
+		)
+		(pad "1" thru_hole circle
+			(at 0 2.4)
+			(size 0.8 0.8)
+			(drill 0.5)
+			(layers "*.Cu" "*.Mask")
+			(remove_unused_layers no)
+			(net 1 "GND")
+			(zone_connect 2)
+		)
+		(pad "1" thru_hole circle
+			(at 1.697056 -1.697056)
+			(size 0.8 0.8)
+			(drill 0.5)
+			(layers "*.Cu" "*.Mask")
+			(remove_unused_layers no)
+			(net 1 "GND")
+			(zone_connect 2)
+		)
+		(pad "1" thru_hole circle
+			(at 1.697056 1.697056)
+			(size 0.8 0.8)
+			(drill 0.5)
+			(layers "*.Cu" "*.Mask")
+			(remove_unused_layers no)
+			(net 1 "GND")
+			(zone_connect 2)
+		)
+		(pad "1" thru_hole circle
+			(at 2.4 0)
+			(size 0.8 0.8)
+			(drill 0.5)
+			(layers "*.Cu" "*.Mask")
+			(remove_unused_layers no)
+			(net 1 "GND")
+			(zone_connect 2)
+		)
 		(embedded_fonts no)
 	)

Commit message: CN2 labels and attribution
Parts:
- CN2: value Neo128 -> C128
Other:
- board text added: "40/80"
- board text added: "CAPLK"
- board text added: "COL0"
- board text added: "COL1"
- board text added: "COL10"
- board text added: "COL2"
- board text added: "COL3"
- board text added: "COL4"
- board text added: "COL5"
- board text added: "COL6"
- board text added: "COL7"
- board text added: "COL8"
- board text added: "COL9"
- board text added: "GND"
- board text added: "Original design by Johan Grip (c128.se) Modified for The C128 Keyboard Project by Jeff Flitton (jeff@flitton.dev) codeberg.org/jflitton/the-c128-keyboard-project"
- board text added: "Plate Ground"
- board text added: "ROW0"
- board text added: "ROW1"
- board text added: "ROW2"
- board text added: "ROW3"
- board text added: "ROW4"
- board text added: "ROW5"
- board text added: "ROW6"
- board text added: "ROW7"
- board text added: "RSTO"
- board text added: "VCC"
