File: plate/pcb_version/plate-6.25u-mx.kicad_pcb (KiCad board)
At the start: 2 copper layers, 401.5 x 137.8 mm, 0 parts

Commit message: fix the plate for MX spacebar. This PCB is untested.
Other:
- outline, holes or cut-outs redrawn
- board text added: "C128 keyboard plate rev 3 (6.25u spacebar, MX caps, 100 mm stabs) - 1.5 mm aluminum PCB - the-c128-keyboard-project"
- board text removed: "C128 keyboard plate rev 3 (stock 9u spacebar) - 1.5 mm aluminum PCB - the-c128-keyboard-project"
